File: hardware/TempSens.kicad_sch (KiCad schematic)
At the start: 20 parts, among them IC1 UCC12040DVE, J1 Conn_01x04_Pin, U1 LM1117-Q1, U2 LM1117-Q1, U3 XISO6463DWR, U4 XISO6463DWR

Commit message: Docs update
Other:
- note removed: "POSTOJI GRESKA SA NAPAJANJEM"
- note removed: "TREBA ODREDITI KOLIKI OSIGURAC JE POTREBAN"
