File: hardware/adc_rc.kicad_sch (KiCad schematic)
At the start: 50 parts, among them J4 Conn_01x08_Pin, J5 Conn_01x08_Pin, J6 Conn_01x08_Pin, U7 ADS114S08B

Commit message: Docs update
Parts:
- R13, R14, R22, R23, R26, R27, R30, R31, R4, R5, R9: value 4.7k -> 680
Connections:
- net +3.3V renamed +3V3_ISO
Other:
- moved on the sheet: C25, C26, C27, C28, C29, C30, C31, C32, C33, C34, C35, C36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
